File: kicad/ESCnix_rev-a/ESCnix.kicad_pcb (KiCad board)
At the start: 2 copper layers, 53 parts, among them J1 INPUT_POWER, Q1 TM60N03DF, Q2 TM60N03DF, Q3 TM60N03DF, Q4 TM60N03DF, Q5 TM60N03DF, Q6 TM60N03DF, U1 EFM8BB21F16G-C-QFN20, U3 AP63203WU-7, U4 FD6288Q

Commit message: Schematic close to complete! Started layout
Parts:
- added C20: 0.1uF, custom:C_0402_1005Metric_NoSilk, F.Cu at (136.7, 113.9)
- added C22: 100nF, custom:C_0402_1005Metric_NoSilk, F.Cu at (141.6, 117.1)
- added C23: 10uF, custom:C_0603_1608Metric_NoSilk, F.Cu at (128.7, 119.7)
- added C25: 10uF, custom:C_0603_1608Metric_NoSilk, F.Cu at (139.1, 95.9)
- added C26: 10uF, custom:C_0603_1608Metric_NoSilk, F.Cu at (137.9, 95.9)
- added C8: 10uF, custom:C_0603_1608Metric_NoSilk, F.Cu at (134.6, 96.0)
- added L2: 4.7uH, Inductor_SMD:L_0402_1005Metric, F.Cu at (141.6, 119.0)
- added R21: 0.5m, Resistor_SMD:R_2512_6332Metric, F.Cu at (134.4, 119.8)
- added U2: EFM8BB21F16G-C-QFN20, easyeda2kicad:QFN-20_L3.0-W3.0-P0.50-BL-EP1.7_EFM8BB21F16G, F.Cu at (133.6, 109.6)
- added U5: AP63203WU-7, Package_TO_SOT_SMD:TSOT-23-6, F.Cu at (139.0, 117.8)
- C1: value 4.7uF -> 0.1uF
- C10, C11: value 1uF -> 10uF; footprint custom:C_0402_1005Metric_NoSilk -> custom:C_0603_1608Metric_NoSilk
- C12: value 0.1uF -> 22uF; footprint custom:C_0402_1005Metric_NoSilk -> custom:C_0805_2012Metric_NoSilk
- C13: value 47uF -> 1uF
- C14: value 1uF -> 4.7uF
- C15: value 1uF -> 0.1uF
- C16, C7: value 0.1uF -> 10uF; footprint custom:C_0402_1005Metric_NoSilk -> custom:C_0603_1608Metric_NoSilk
- C17: value 47uF -> 100nF
- C18, C19: value 1uF -> 22uF; footprint custom:C_0402_1005Metric_NoSilk -> custom:C_0805_2012Metric_NoSilk
- C3: value 10uF -> 0.1uF; footprint custom:C_0603_1608Metric_NoSilk -> custom:C_0402_1005Metric_NoSilk
- C4: value 22uF -> 10uF
- C5: value 100nF -> 10uF
- C6: footprint custom:C_0603_1608Metric_NoSilk -> custom:C_0805_2012Metric_NoSilk
- C9: value 47uF -> 10uF; footprint custom:C_0402_1005Metric_NoSilk -> custom:C_0603_1608Metric_NoSilk
- D1: value RED -> RB520S-30; footprint custom:LED_0603_1608Metric_NoSilk -> custom:D_SOD-523_NoSilk
- D2: value BLUE -> RB520S-30; footprint custom:LED_0603_1608Metric_NoSilk -> custom:D_SOD-523_NoSilk
- D3: value GREEN -> RB520S-30; footprint custom:LED_0603_1608Metric_NoSilk -> custom:D_SOD-523_NoSilk
- D4: value RB520S-30 -> RED; footprint Diode_SMD:D_SOD-523 -> custom:LED_0603_1608Metric_NoSilk
- D5: value RB520S-30 -> BLUE; footprint Diode_SMD:D_SOD-523 -> custom:LED_0603_1608Metric_NoSilk
- D6: value RB520S-30 -> GREEN; footprint Diode_SMD:D_SOD-523 -> custom:LED_0603_1608Metric_NoSilk
- R10: value 4R7 -> 12k
- R13, R7: value 12k -> 100k
- R14, R15, R9: value 4R7 -> 100k
- R16: value 100k -> 1k
- R17, R18: value 12k -> 1k
- R2, R3, R4: value 1k -> 4R7
- R6: value 100k -> 4R7
- U1: value EFM8BB21F16G-C-QFN20 -> FD6288Q; footprint easyeda2kicad:QFN-20_L3.0-W3.0-P0.50-BL-EP1.7_EFM8BB21F16G -> easyeda2kicad:QFN-24_L4.0-W4.0-P0.50-BL-EP2.6
- U4: value FD6288Q -> INA180A3IDBVR; footprint easyeda2kicad:QFN-24_L4.0-W4.0-P0.50-BL-EP2.6 -> Package_TO_SOT_SMD:SOT-23-5
- moved C16 24.6 mm to (139.0, 120.1)
- moved J1 23.6 mm to (133.4, 125.0), turned to 90 degrees
- moved C17 21.5 mm to (131.2, 116.5), turned to -90 degrees
- moved C12 20.1 mm to (127.8, 114.3), turned to 90 degrees
- moved L1 16.8 mm to (131.2, 118.9), turned to -90 degrees
- moved C18 15.5 mm to (140.2, 114.2), turned to 90 degrees
- moved R6 14.5 mm to (137.9, 98.4), turned to 90 degrees
- moved C19 14.0 mm to (138.3, 114.2), turned to 90 degrees
- moved R11 13.5 mm to (139.8, 104.8)
- moved C14 13.3 mm to (128.7, 109.9)
- moved C15 13.3 mm to (128.7, 111.5)
- moved R12 13.3 mm to (139.8, 105.7)
- moved R15 13.2 mm to (139.8, 104.0)
- moved C6 13.1 mm to (129.6, 114.3), turned to 90 degrees
- moved R16 13.0 mm to (137.3, 107.7)
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Connections:
- C1 pad 1: +3V3 -> VB1
- C1 pad 2: GND -> PHASE_A
- C10 pad 1: VCC -> VBAT
- C11 pad 1: VCC -> VBAT
- C12 pad 1: VB2 -> +3V3
- C12 pad 2: PHASE_B -> GND
- C14 pad 1: VCC -> +3V3
- C15 pad 1: VCC -> +3V3
- C16 pad 1: VB3 -> VCC
- C16 pad 2: PHASE_C -> GND
- C17 pad 1: VCC -> Net-(U3-BST)
- C17 pad 2: GND -> Net-(U3-SW)
- C18 pad 1: VCC -> +5V
- C19 pad 1: VCC -> +5V
- C2 pad 1: +3V3 -> VB2
- C2 pad 2: GND -> PHASE_B
- C3 pad 1: VCC -> VB3
- C3 pad 2: GND -> PHASE_C
- C4 pad 1: +3V3 -> VBAT
- C5 pad 1: Net-(U3-BST) -> VBAT
- C5 pad 2: Net-(U3-SW) -> GND
- C7 pad 1: VB1 -> VBAT
- C7 pad 2: PHASE_A -> GND
- C9 pad 1: VCC -> VBAT
- D1 pad 1: GND -> VB1
- D1 pad 2: Net-(D1-A) -> +5V
- D2 pad 1: GND -> VB2
- D2 pad 2: Net-(D2-A) -> +5V
- D3 pad 1: GND -> VB3
- D3 pad 2: Net-(D3-A) -> +5V
- D4 pad 1: VB1 -> GND
- D4 pad 2: VCC -> Net-(D4-A)
- D5 pad 1: VB2 -> GND
- D5 pad 2: VCC -> Net-(D5-A)
- D6 pad 1: VB3 -> GND
- D6 pad 2: VCC -> Net-(D6-A)
- Q1 pad 1: GND -> PHASE_A
- Q1 pad 2: GND -> PHASE_A
- Q1 pad 3: GND -> PHASE_A
- Q1 pad 5: PHASE_A -> VBAT
- Q2 pad 1: PHASE_A -> GND
- Q2 pad 2: PHASE_A -> GND
- Q2 pad 3: PHASE_A -> GND
- Q2 pad 5: VCC -> PHASE_A
- Q3 pad 5: VCC -> VBAT
- Q5 pad 5: VCC -> VBAT
- R1 pad 2: Net-(Q2-G) -> Net-(Q1-G)
- R10 pad 1: LO2 -> B_MEASURE
- R10 pad 2: Net-(Q4-G) -> GND
- R11 pad 1: PHASE_B -> PHASE_C
- R11 pad 2: B_MEASURE -> C_MEASURE
- R12 pad 1: B_MEASURE -> C_MEASURE
- R13 pad 1: B_MEASURE -> A_MEASURE
- R14 pad 1: HO3 -> B_MEASURE
- R14 pad 2: Net-(Q5-G) -> NEUTRAL
- R15 pad 1: LO3 -> C_MEASURE
- R15 pad 2: Net-(Q6-G) -> NEUTRAL
- R16 pad 1: PHASE_C -> Net-(D4-A)
- R16 pad 2: C_MEASURE -> LED_RED
- R17 pad 1: C_MEASURE -> Net-(D5-A)
- R17 pad 2: GND -> LED_BLUE
- R18 pad 1: C_MEASURE -> Net-(D6-A)
- R18 pad 2: NEUTRAL -> LED_GREEN
- R2 pad 1: Net-(D1-A) -> LO1
- R2 pad 2: LED_RED -> Net-(Q2-G)
- R3 pad 1: Net-(D2-A) -> HO2
- R3 pad 2: LED_BLUE -> Net-(Q3-G)
- R4 pad 1: Net-(D3-A) -> LO2
- R4 pad 2: LED_GREEN -> Net-(Q4-G)
- R5 pad 1: LO1 -> HO3
- R5 pad 2: Net-(Q1-G) -> Net-(Q5-G)
- R6 pad 1: PHASE_A -> LO3
- R6 pad 2: A_MEASURE -> Net-(Q6-G)
- R7 pad 1: A_MEASURE -> PHASE_A
- R7 pad 2: GND -> A_MEASURE
- R8 pad 2: NEUTRAL -> GND
- R9 pad 1: HO2 -> PHASE_B
- R9 pad 2: Net-(Q3-G) -> B_MEASURE
- U1 pad 1: unconnected-(U1-P0.1-Pad1) -> C_COM
- U1 pad 10: unconnected-(U1-P1.3-Pad10) -> LO2
- U1 pad 11: unconnected-(U1-P1.2-Pad11) -> LO1
- U1 pad 12: GND -> PHASE_C
- U1 pad 13: unconnected-(U1-P1.1-Pad13) -> HO3
- U1 pad 14: unconnected-(U1-P1.0-Pad14) -> VB3
- U1 pad 15: unconnected-(U1-P0.7-Pad15) -> PHASE_B
- U1 pad 16: unconnected-(U1-P0.6-Pad16) -> HO2
- U1 pad 17: unconnected-(U1-P0.5-Pad17) -> VB2
- U1 pad 18: unconnected-(U1-P0.4-Pad18) -> PHASE_A
- U1 pad 19: unconnected-(U1-P0.3-Pad19) -> HO1
- U1 pad 2: unconnected-(U1-P0.0-Pad2) -> B_COM
- U1 pad 20: unconnected-(U1-P0.2-Pad20) -> VB1
- U1 pad 21: GND -> unconnected-(U1-NC-Pad21)
- U1 pad 3: GND -> A_COM
- U1 pad 4: +3V3 -> VCC
- U1 pad 6: unconnected-(U1-P2.0/C2D-Pad6) -> GND
- U1 pad 9: unconnected-(U1-P1.4-Pad9) -> LO3
- U4 pad 1: C_COM -> CURR_SENSE
- U4 pad 2: B_COM -> GND
- U4 pad 3: A_COM -> VCC
- U4 pad 4: VCC -> VBAT
- U4 pad 5: unconnected-(U4-NC-Pad5) -> +3.3V
Routing:
- net VBAT: track 0.00 -> 24.5 mm, vias 0 -> 12
- net Net-(Q6-G): track 0.00 -> 11.1 mm, vias 0 -> 2
- net Net-(Q4-G): track 0.00 -> 11.0 mm, vias 0 -> 2
- net Net-(Q2-G): track 0.00 -> 10.6 mm, vias 0 -> 2
- net Net-(Q3-G): track 0.00 -> 9.24 mm, vias 0 -> 2
- net Net-(Q5-G): track 0.00 -> 9.24 mm, vias 0 -> 2
- net Net-(Q1-G): track 0.00 -> 8.38 mm, vias 0 -> 2
- net PHASE_C: track 0.00 -> 6.29 mm
- net PHASE_A: track 0.00 -> 6.24 mm
- net PHASE_B: track 0.00 -> 6.09 mm
- net GND: track 0.00 -> 2.36 mm, vias 0 -> 2
- added copper zone on B.Cu, net GND
- added copper zone on F.Cu, net GND
- added copper zone on In1.Cu, net GND
- added copper zone on F.Cu, net VBAT
- added copper zone on In2.Cu, net VBAT
Other:
- copper layers 2 -> 4

Commit message: Initial layout done, started routing a bit
Parts:
- added J2: SWD, custom:Conn_3_2_SMD, F.Cu at (129.2, 103.0)
- added J4: Conn_01x01, custom:Conn_1_BigPad, F.Cu at (138.9, 121.6)
- added J5: SWD, custom:Conn_3_Accesory2, F.Cu at (133.2, 122.3)
- added J6: Conn_01x01, custom:Conn_1_Accesory2, F.Cu at (126.3, 118.7)
- J1: value INPUT_POWER -> Conn_01x01; footprint custom:Conn_2_Bat -> custom:Conn_1_BigPad
- moved D4 14.3 mm to (127.0, 113.5), turned to 90 degrees
- moved D6 12.1 mm to (128.2, 108.7)
- moved D5 11.8 mm to (128.2, 110.1)
- moved R16 11.1 mm to (126.9, 111.5)
- moved C22 10.7 mm to (131.1, 119.0), turned to 90 degrees
- moved R8 10.6 mm to (138.0, 105.6), turned to 180 degrees
- moved R13 10.6 mm to (137.7, 109.1), turned to -90 degrees
- moved C19 9.64 mm to (129.8, 118.6), turned to -90 degrees
- moved R7 9.51 mm to (138.0, 106.5)
- moved R10 9.44 mm to (138.0, 103.9), turned to 180 degrees
- moved R14 9.43 mm to (138.5, 109.1), turned to -90 degrees
- moved L2 9.12 mm to (132.6, 120.5), turned to 0 degrees
- moved R9 8.79 mm to (138.0, 104.8)
- moved C14 8.11 mm to (136.8, 109.1), turned to -90 degrees
- moved L1 7.81 mm to (128.7, 111.5), turned to 180 degrees
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Connections:
- J1 pad 1: VCC -> GND
- U2 pad 1: unconnected-(U2-P0.1-Pad1) -> A_MEASURE
- U2 pad 10: unconnected-(U2-P1.3-Pad10) -> B_COM
- U2 pad 11: unconnected-(U2-P1.2-Pad11) -> B_PWM
- U2 pad 13: unconnected-(U2-P1.1-Pad13) -> A_COM
- U2 pad 14: unconnected-(U2-P1.0-Pad14) -> A_PWM
- U2 pad 15: unconnected-(U2-P0.7-Pad15) -> LED_GREEN
- U2 pad 16: unconnected-(U2-P0.6-Pad16) -> LED_BLUE
- U2 pad 17: unconnected-(U2-P0.5-Pad17) -> RTX
- U2 pad 19: unconnected-(U2-P0.3-Pad19) -> C_MEASURE
- U2 pad 2: unconnected-(U2-P0.0-Pad2) -> NEUTRAL
- U2 pad 20: unconnected-(U2-P0.2-Pad20) -> B_MEASURE
- U2 pad 7: unconnected-(U2-P1.6-Pad7) -> LED_RED
- U2 pad 8: unconnected-(U2-P1.5-Pad8) -> C_COM
- U2 pad 9: unconnected-(U2-P1.4-Pad9) -> C_PWM
Routing:
- net PHASE_A: track 6.24 -> 38.0 mm, vias 0 -> 4
- net PHASE_B: track 6.09 -> 35.6 mm, vias 0 -> 4
- net PHASE_C: track 6.29 -> 29.9 mm, vias 0 -> 3
- net C_MEASURE: track 0.00 -> 16.8 mm, vias 0 -> 2
- net LED_RED: track 0.00 -> 15.1 mm, vias 0 -> 2
- net GND: track 2.36 -> 16.4 mm, vias 2 -> 3
- net B_MEASURE: track 0.00 -> 13.4 mm, vias 0 -> 2
- net C2CK: track 0.00 -> 11.8 mm, vias 0 -> 2
- net C2CD: track 0.00 -> 11.7 mm, vias 0 -> 2
- net LO1: track 0.00 -> 10.3 mm, vias 0 -> 2
- net A_PWM: track 0.00 -> 8.18 mm
- net A_COM: track 0.00 -> 8.06 mm, vias 0 -> 2
- net A_MEASURE: track 0.00 -> 8.06 mm, vias 0 -> 2
- net LO2: track 0.00 -> 7.95 mm, vias 0 -> 2
- net LO3: track 0.00 -> 6.84 mm, vias 0 -> 2
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