File: kicad/ESCnix_rev-a/ESCnix.kicad_sch (KiCad schematic)
At the start: 54 parts, among them J1 INPUT_POWER, Q1 TM60N03DF, Q2 TM60N03DF, Q3 TM60N03DF, Q4 TM60N03DF, Q5 TM60N03DF, Q6 TM60N03DF, U1 FD6288Q, U2 EFM8BB21F16G-C-QFN20, U3 AP63203WU-7

Commit message: Schematic close to complete! Started layout
Parts:
- added C20: 0.1uF, custom:C_0402_1005Metric_NoSilk, symbol Device:C_Small
- added C22: 100nF, custom:C_0402_1005Metric_NoSilk, symbol Device:C_Small
- added C23, C25, C26: 10uF, custom:C_0603_1608Metric_NoSilk, symbol Device:C_Small
- added J2: SWD, symbol Connector_Generic:Conn_01x03
- added J3: COM, symbol Connector_Generic:Conn_01x04
- added L2: 4.7uH, Inductor_SMD:L_0402_1005Metric, symbol Device:L_Small
- added R21: 0.5m, Resistor_SMD:R_2512_6332Metric, symbol Device:R_Small
- added TP1, TP2, TP3, TP4, TP5: TestPoint, symbol Connector:TestPoint
- added U4: INA180A3IDBVR, Package_TO_SOT_SMD:SOT-23-5, symbol Amplifier_Current:INA180A3
- added U5: AP63203WU-7, Package_TO_SOT_SMD:TSOT-23-6, symbol Regulator_Switching:AP63203WU
- C10, C11, C7, C8, C9: value 1uF -> 10uF; footprint custom:C_0402_1005Metric_NoSilk -> custom:C_0603_1608Metric_NoSilk; LCSC Part (none) -> C96446
- C12: value 1uF -> 22uF; footprint custom:C_0402_1005Metric_NoSilk -> custom:C_0805_2012Metric_NoSilk; LCSC Part (none) -> C45783
- C13: footprint (none) -> custom:C_0402_1005Metric_NoSilk
- C16: LCSC Part (none) -> C96446
- C17: footprint custom:C_0603_1608Metric_NoSilk -> custom:C_0402_1005Metric_NoSilk
- C18, C19: footprint custom:C_0603_1608Metric_NoSilk -> custom:C_0805_2012Metric_NoSilk; LCSC Part (none) -> C45783
- C4, C5: value 47uF -> 10uF; footprint custom:C_0402_1005Metric_NoSilk -> custom:C_0603_1608Metric_NoSilk; LCSC Part (none) -> C96446
- C6: value 47uF -> 22uF; footprint custom:C_0402_1005Metric_NoSilk -> custom:C_0805_2012Metric_NoSilk; LCSC Part (none) -> C45783
- D1, D2, D3: footprint Diode_SMD:D_SOD-523 -> custom:D_SOD-523_NoSilk
- R13, R14, R15: value 12k -> 100k
Connections:
- net +3V3: now also C12.1, C6.1, TP1.1; no longer C18.1, C19.1
- net A_MEASURE: now also TP3.1
- net B_MEASURE: now also TP4.1
- net C2CD: now also U2.6 (P2.0/C2D), J2.2 (Pin_2)
- net C2CK: now also U2.5 (RSTB/C2CK), J2.1 (Pin_1)
- net C_MEASURE: now also TP5.1
- net GND: now also U1.25 (EP), C20.2, C23.2, C25.2, C26.2, J2.3 (Pin_3), J3.4 (Pin_4), U4.2 (GND), U5.4 (GND)
- net NEUTRAL: now also TP2.1
- net RTX: now also J3.2 (Pin_2)
- net VCC: now also C23.1, R21.1, U4.3 (+), U5.2 (EN), U5.3 (IN); no longer C10.1, C11.1, C12.1, C4.1, C5.1, C6.1, C7.1, C8.1, C9.1, D1.2 (A), D2.2 (A), D3.2 (A), Q1.5 (D), Q3.5 (D), Q5.5 (D)
- new net: C22.1, U5.6 (BST)
- new net: C22.2, L2.1, U5.5 (SW)
- new net +3.3V: C20.1, U4.5 (V+)
- new net +5V: C18.1, C19.1, D1.2 (A), D2.2 (A), D3.2 (A), J3.3 (Pin_3), L2.2, U5.1 (FB)
- new net CURR_SENSE: J3.1 (Pin_1), U4.1
- new net VBAT: C10.1, C11.1, C25.1, C26.1, C4.1, C5.1, C7.1, C8.1, C9.1, Q1.5 (D), Q3.5 (D), Q5.5 (D), R21.2, U4.4 (-)
Other:
- note added: "Current measurement"
- note added: "Max current: 60A -> Max voltage: 30mV -> Max power: 1.8W Gain: 100 ADC max: 3V"
- moved on the sheet: J1

Commit message: Initial layout done, started routing a bit
Parts:
- removed J1: INPUT_POWER, custom:Conn_2_Bat, symbol Connector_Generic:Conn_01x02
- removed J3: COM, symbol Connector_Generic:Conn_01x04
- added J1, J4: Conn_01x01, custom:Conn_1_BigPad, symbol Connector_Generic:Conn_01x01
- added J5: SWD, custom:Conn_3_Accesory2, symbol Connector_Generic:Conn_01x03
- added J6: Conn_01x01, custom:Conn_1_Accesory2, symbol Connector_Generic:Conn_01x01
- J2: footprint (none) -> custom:Conn_3_2_SMD
Connections:
- net +5V: now also J5.2 (Pin_2)
- net A_COM: now also U2.13 (P1.1)
- net A_MEASURE: now also U2.1 (P0.1)
- net A_PWM: now also U2.14 (P1.0)
- net B_COM: now also U2.10 (P1.3)
- net B_MEASURE: now also U2.20 (P0.2)
- net B_PWM: now also U2.11 (P1.2)
- net C2CK: now also J2.3 (Pin_3); no longer J2.1 (Pin_1)
- net CURR_SENSE: now also J6.1 (Pin_1)
- net C_COM: now also U2.8 (P1.5)
- net C_MEASURE: now also U2.19 (P0.3)
- net C_PWM: now also U2.9 (P1.4)
- net GND: now also J2.1 (Pin_1), J1.1 (Pin_1), J5.3 (Pin_3); no longer J2.3 (Pin_3)
- net LED_BLUE: now also U2.16 (P0.6)
- net LED_GREEN: now also U2.15 (P0.7)
- net LED_RED: now also U2.7 (P1.6)
- net NEUTRAL: now also U2.2 (P0.0)
- net RTX: now also U2.17 (P0.5), J5.1 (Pin_1)
- net VCC: now also J4.1 (Pin_1)
- no-connect marks 4 -> 5
Other:
- note added: "E.inc"
